File: ITFA-CUBE-ING-V00.kicad_sch (KiCad schematic)
At the start: 34 parts, among them J1 Conn_01x04, U1 STM32H743VITx, U2 W25Q128JVS, Y1 25MHz 10pF, Y2 32.768K 7pF

Commit message: Avance uc
Parts:
- removed J1: Conn_01x04, Connector_PinHeader_2.54mm:PinHeader_1x04_P2.54mm_Horizontal, symbol Connector_Generic:Conn_01x04
- added J1: Conn_02x04_Odd_Even, Connector_PinHeader_2.54mm:PinHeader_2x04_P2.54mm_Horizontal, symbol Connector_Generic:Conn_02x04_Odd_Even
- added SW1: SW_DIP_x10, symbol Switch:SW_DIP_x10
Connections:
- net SPI_Flash_CLK is gone; now on net SPI1_CLK: U2.6 (CLK)
- net SPI_Flash_CS is gone; now on net SPI1_Flash1_CS: R3.1, U2.1 (~{CS})
- net SPI_Flash_MISO is gone; now on net SPI1_MISO: U2.2 (DO/IO_{1})
- net SPI_Flash_MOSI is gone; now on net SPI1_MOSI: U2.5 (DI/IO_{0})
- net +3.3V: now also J1.2 (Pin_2)
- net GND: now also J1.7 (Pin_7), J1.8 (Pin_8)
- net SWCLK: now also J1.6 (Pin_6)
- net SWDIO: now also J1.4 (Pin_4)
- net RCC_OSC32_OUT: now reaches C3.1, U1.9 (PC15), Y2.1
- net RCC_OSC32_IN: now reaches C4.1, U1.8 (PC14), Y2.2
- net SPI4_CLK: now reaches U1.1 (PE2)
- net SPI4_CLK: now also SW1.5
- net USART2_TX: now reaches U1.24 (PA2)
- net USART2_TX: now also SW1.1
- net USART2_RX: now reaches U1.25 (PA3)
- net USART2_RX: now also SW1.2
- net SPI1_Flash1_CS: now reaches U1.28 (PA4)
- net SPI1_CLK: now reaches U1.29 (PA5)
- net SPI1_MISO: now reaches U1.30 (PA6)
- net SPI1_MOSI: now reaches U1.31 (PA7)
- net SPI4_MISO: now reaches U1.4 (PE5)
- net SPI4_MISO: now also SW1.6
- net I2C2_SCL: now reaches U1.46 (PB10)
- net I2C2_SCL: now also SW1.3
- net I2C2_SDA: now reaches U1.47 (PB11)
- net I2C2_SDA: now also SW1.4
- net SPI4_MOSI: now reaches U1.5 (PE6)
- net SPI4_MOSI: now also SW1.7
- net USART1_TX: now reaches U1.68 (PA9)
- net USART1_TX: now also J1.1 (Pin_1)
- net USART1_RX: now reaches U1.69 (PA10)
- net USART1_RX: now also J1.3 (Pin_3)
- net SWO: now reaches U1.89 (PB3)
- net SWO: now also J1.5 (Pin_5)
- net I2C1_SCL: now reaches U1.92 (PB6)
- net I2C1_SDA: now reaches U1.93 (PB7)
- net CAN1_ RD renamed CAN1-
- net CAN1_ TD renamed CAN1+
- net CAN_1_N: no longer names the net of H1.24 (Pin_24)
- net CAN_1_P: no longer names the net of H1.23 (Pin_23)
- net CAN_2_N: no longer names the net of H2.24 (Pin_24)
- net CAN_2_P: no longer names the net of H2.23 (Pin_23)
- net CPU_MODE: no longer names the net of H1.30 (Pin_30)
- net CPU_WD_1: no longer names the net of H1.27 (Pin_27)
- net GLO_FAULT: no longer names the net of H1.26 (Pin_26)
- net GLO_KS_1: no longer names the net of H1.35 (Pin_35)
- net GLO_SYNC: no longer names the net of H1.25 (Pin_25)
- net I2C_1_SCL: no longer names the net of H1.21 (Pin_21)
- net I2C_1_SDA: no longer names the net of H1.22 (Pin_22)
- net I2C_2_SCL: no longer names the net of H2.21 (Pin_21)
- net I2C_2_SDA: no longer names the net of H2.22 (Pin_22)
- net SPI_1_CS1: no longer names the net of H1.9 (Pin_9)
- net SPI_1_CS2: no longer names the net of H1.7 (Pin_7)
- net SPI_1_MISO: no longer names the net of H1.12 (Pin_12)
- net SPI_1_MOSI: no longer names the net of H1.10 (Pin_10)
- net SPI_1_SCK: no longer names the net of H1.11 (Pin_11)
- net SPI_2_CS1: no longer names the net of H2.9 (Pin_9)
- net SPI_2_CS2: no longer names the net of H2.7 (Pin_7)
- net SPI_2_MISO: no longer names the net of H2.12 (Pin_12)
- net SPI_2_MOSI: no longer names the net of H2.10 (Pin_10)
- net SPI_2_SCK: no longer names the net of H2.11 (Pin_11)
- net SUP_3V3: no longer names the net of H2.27 (Pin_27)
- net SUP_3V3: no longer H2.28 (Pin_28)
- net SUP_5V: no longer names the net of H2.25 (Pin_25)
- net SUP_5V: no longer H2.26 (Pin_26)
- net UART_1_CTS: no longer names the net of H1.14 (Pin_14)
- net UART_1_RST: no longer names the net of H1.16 (Pin_16)
- net UART_1_RX: no longer names the net of H1.15 (Pin_15)
- net UART_1_TX: no longer names the net of H1.13 (Pin_13)
- net UART_2_CTS: no longer names the net of H2.14 (Pin_14)
- net UART_2_RST: no longer names the net of H2.16 (Pin_16)
- net UART_2_RX: no longer names the net of H2.15 (Pin_15)
- net UART_2_TX: no longer names the net of H2.13 (Pin_13)
- net UART_RCS_1_CTS: no longer names the net of H1.18 (Pin_18)
- net UART_RCS_1_RST: no longer names the net of H1.20 (Pin_20)
- net UART_RCS_1_RX: no longer names the net of H1.19 (Pin_19)
- net UART_RCS_1_TX: no longer names the net of H1.17 (Pin_17)
- net UART_RCS_2_CTS: no longer names the net of H2.18 (Pin_18)
- net UART_RCS_2_RST: no longer names the net of H2.20 (Pin_20)
- net UART_RCS_2_RX: no longer names the net of H2.19 (Pin_19)
- net UART_RCS_2_TX: no longer names the net of H2.17 (Pin_17)
- net USER_1_1: no longer names the net of H1.5 (Pin_5)
- net USER_1_2: no longer names the net of H1.6 (Pin_6)
- net USER_1_4: no longer names the net of H1.8 (Pin_8)
- net USER_2_1: no longer names the net of H2.5 (Pin_5)
- net USER_2_2: no longer names the net of H2.6 (Pin_6)
- net USER_2_4: no longer names the net of H2.8 (Pin_8)
- net USER_3_1: no longer names the net of H1.39 (Pin_39)
- net USER_3_2: no longer names the net of H1.40 (Pin_40)
- net USER_3_3: no longer names the net of H1.41 (Pin_41)
- net USER_3_4: no longer names the net of H1.42 (Pin_42)
- net USER_4_1: no longer names the net of H2.39 (Pin_39)
- net USER_4_2: no longer names the net of H2.40 (Pin_40)
- net USER_4_3: no longer names the net of H2.41 (Pin_41)
- net USER_4_4: no longer names the net of H2.42 (Pin_42)
- net USER_5_1: no longer names the net of H1.43 (Pin_43)
- net USER_5_2: no longer names the net of H1.44 (Pin_44)
- net USER_5_3: no longer names the net of H1.45 (Pin_45)
- net USER_5_4: no longer names the net of H1.46 (Pin_46)
- net USER_6_1: no longer names the net of H2.43 (Pin_43)
- net USER_6_2: no longer names the net of H2.44 (Pin_44)
- net USER_6_3: no longer names the net of H2.47 (Pin_47)
- net USER_6_4: no longer names the net of H2.48 (Pin_48)
Other:
- note added: "Prog. Debug + UART"
- company: (none) -> Instituto Argentino de Radioastronomia
- title: (none) -> STM32 Test Board
- moved on the sheet: C1, C19, C2, H1, MH1, MH2, MH3, MH4, R3, U2, Y1

Commit message: Actualizandon esquematico
Parts:
- added SW2: SW_DIP_x10, symbol Switch:SW_DIP_x10
Connections:
- net +3.3V: now also H2.46 (Pin_46)
- net GND: now also H1.29 (Pin_29), H1.30 (Pin_30), H1.31 (Pin_31), H1.32 (Pin_32), H2.33 (Pin_33), H2.34 (Pin_34), H2.35 (Pin_35), H2.36 (Pin_36); no longer H1.33 (Pin_33), H2.29 (Pin_29), H2.30 (Pin_30), H2.32 (Pin_32)
- net SPI4_MISO: now also SW1.7; no longer SW1.6
- net SPI4_MOSI: now also SW1.8; no longer SW1.7
- net CAN_A_L: now reaches H2.1 (Pin_1)
- net SPI_A_MOSI: now reaches H2.10 (Pin_10)
- net SPI_A_MOSI: now also SW1.13
- net SPI_A_CLK: now reaches H2.11 (Pin_11)
- net SPI_A_CLK: now also SW1.16
- net SPI_A_MISO: now reaches H2.12 (Pin_12)
- net SPI_A_MISO: now also SW1.14
- net UART_A_TX: now reaches H2.13 (Pin_13)
- net UART_A_TX: now also SW1.20
- net UART_A_RX: now reaches H2.15 (Pin_15)
- net UART_A_RX: now also SW1.19
- net CAN_B_L: now reaches H2.2 (Pin_2)
- net I2C_B_SCL: now reaches H2.21 (Pin_21)
- net UART_B_TX: now reaches H2.22 (Pin_22)
- net I2C_B_SDA: now reaches H2.23 (Pin_23)
- net UART_B_RX: now reaches H2.24 (Pin_24)
- net +5V: now reaches H2.25 (Pin_25)
- net +5V: now also H1.25 (Pin_25), H1.26 (Pin_26), H2.26 (Pin_26)
- net CAN_A_H: now reaches H2.3 (Pin_3)
- net CAN_B_H: now reaches H2.4 (Pin_4)
- net I2C_A_SDA: now reaches H2.41 (Pin_41)
- net I2C_A_SDA: now also SW1.17
- net I2C_A_SCL: now reaches H2.43 (Pin_43)
- net I2C_A_SCL: now also SW1.18
- net ENA_PWR_1: now reaches H2.45 (Pin_45)
- net ENA_PWR_2: now reaches H2.47 (Pin_47)
- net PWR_2: now reaches H2.48 (Pin_48)
- net ENA_PWR_3: now reaches H2.49 (Pin_49)
- net UART_C_TX: now reaches H2.5 (Pin_5)
- net PWR_3: now reaches H2.50 (Pin_50)
- net ENA_PWR_4: now reaches H2.51 (Pin_51)
- net PWR_4: now reaches H2.52 (Pin_52)
- net UART_D_TX: now reaches H2.6 (Pin_6)
- net UART_C_RX: now reaches H2.7 (Pin_7)
- net UART_D_RX: now reaches H2.8 (Pin_8)
- net SPI_A_CS: now reaches H2.9 (Pin_9)
- net SPI_A_CS: now also SW1.15
- net DIG_A_01: now reaches H1.1 (Pin_1)
- net DIG_A_01: now also SW2.20
- net DIG_A_10: now reaches H1.10 (Pin_10)
- net DIG_A_10: now also SW2.11
- net SW2_VBAT: now reaches H1.11 (Pin_11)
- net SW1_VBAT: now reaches H1.12 (Pin_12)
- net DIG_A_02: now reaches H1.2 (Pin_2)
- net DIG_A_02: now also SW2.19
- net DIG_A_03: now reaches H1.3 (Pin_3)
- net DIG_A_03: now also SW2.18
- net PWR_5: now reaches H1.34 (Pin_34)
- net ENA_PWR_6: now reaches H1.35 (Pin_35)
- net PWR_6: now reaches H1.36 (Pin_36)
- net ENA_PWR_7: now reaches H1.37 (Pin_37)
- net PWR_7: now reaches H1.38 (Pin_38)
- net ENA_PWR_8: now reaches H1.39 (Pin_39)
- net DIG_A_04: now reaches H1.4 (Pin_4)
- net DIG_A_04: now also SW2.17
- net PWR_8: now reaches H1.40 (Pin_40)
- net VBAT: now reaches H1.45 (Pin_45)
- net VBAT: now also H1.46 (Pin_46)
- net RBF_OPEN: now reaches H1.49 (Pin_49)
- net DIG_A_05: now reaches H1.5 (Pin_5)
- net DIG_A_05: now also SW2.16
- net RBF_GND: now reaches H1.50 (Pin_50)
- net KS_OPEN: now reaches H1.51 (Pin_51)
- net KS_GND: now reaches H1.52 (Pin_52)
- net DIG_A_06: now reaches H1.6 (Pin_6)
- net DIG_A_06: now also SW2.15
- net DIG_A_07: now reaches H1.7 (Pin_7)
- net DIG_A_07: now also SW2.14
- net DIG_A_08: now reaches H1.8 (Pin_8)
- net DIG_A_08: now also SW2.13
- net DIG_A_09: now reaches H1.9 (Pin_9)
- net DIG_A_09: now also SW2.12
- net SPI4_CS: now reaches U1.2 (PE3)
- net SPI4_CS: now also SW1.6
- net PC4: now reaches U1.32 (PC4)
- net PC4: now also SW2.1
- net PC5: now reaches U1.33 (PC5)
- net PC5: now also SW2.2
- net PC6: now reaches U1.63 (PC6)
- net PC6: now also SW2.3
- net PC7: now reaches U1.64 (PC7)
- net PC7: now also SW2.4
- net PC8: now reaches U1.65 (PC8)
- net PC8: now also SW2.5
- net PC9: now reaches U1.66 (PC9)
- net PC9: now also SW2.6
- net PC13: now reaches U1.7 (PC13)
- net PC13: now also SW2.10
- net PC10: now reaches U1.78 (PC10)
- net PC10: now also SW2.7
- net PC11: now reaches U1.79 (PC11)
- net PC11: now also SW2.8
- net PC12: now reaches U1.80 (PC12)
- net PC12: now also SW2.9
- new net ENA_PWR_5: H1.33 (Pin_33)
- no-connect marks 38 -> 93
Other:
- note added: "BORDE DE PLACA"
- note added: "INTERIOR DE PLACA"
- moved on the sheet: C10, C11, C12, C13, C16, C17, C18, C3, C4, C5, C6, C7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
